Commit message: Added controllers, all sensors, sensible intertia values for chassis and wheels, weights

File: urdf/hokuyo.xacro (robot description, xacro)
@@ -5,5 +5,5 @@
     <link name="${name}">
       <collision>
-        <origin xyz="0 0 0.035" rpy="0 0 0"/>
+      <origin xyz="0 0 -0.0325" rpy="0 0 0"/>
         <geometry>
           <box size="0.05 0.05 0.07"/>
@@ -11,8 +11,4 @@
       </collision>
       <visual>
-<!--          <origin xyz="0 0 0.035" rpy="0 0 0"/>
-          <geometry>
-            <box size="0.05 0.05 0.07"/>
-          </geometry>-->
         <origin xyz="0 0 0" rpy="0 0 0"/>
         <geometry>
@@ -40,12 +36,13 @@
                 <!-- The URG-04LX-UG01  has  683 steps with 0.35139 Degree resolution -->
                 <resolution>1</resolution>
-                <max_angle>2.0944</max_angle> <!-- 120 Degree -->
-                <min_angle>-2.0944</min_angle> <!-- -120 Degree -->
+                <max_angle>2.0944</max_angle> <!-- 120 Degrees -->
+                <min_angle>-2.0944</min_angle> <!-- -120 Degrees -->
                 <samples>683</samples>
               </horizontal>
             </scan>
             <range>
-              <min>0.08</min>
-              <max>5</max>
+              <!-- range is artificially increased in order to prevent the sensor from self-colliding, actually 2cm -->
+              <min>0.05</min>
+              <max>5.6</max>
               <resolution>0.01</resolution>
             </range>
@@ -56,9 +53,6 @@
             <frameName>${name}</frameName>
           </plugin>
-          <!--
-          <plugin name="laser" filename="libRayPlugin.so" />
-          -->
           <always_on>1</always_on>
-          <update_rate>30</update_rate>
+          <update_rate>10</update_rate>
           <visualize>true</visualize>
         </sensor>

File: urdf/pepperl_fuchs_ml100_8_1000_RT.xacro (robot description, xacro)
@@ -7,9 +7,9 @@
             <box size="0.0205 0.011 0.031"/>
         </geometry>-->
-        <origin xyz="0 0 0.01505" rpy="0 0 ${3*PI/2}"/>
+        <origin xyz="0.005125 0.011 0.01505" rpy="0 0 ${3*PI/2}"/>
       </collision>
       <visual>
         <geometry>
-          <mesh filename="package://drive_gazebo_sim/meshes/pepperluchs.dae" scale="0.001 0.001 0.001"/>
+          <mesh filename="package://drive_gazebo_sim/meshes/pepperl_fuchs.dae" scale="0.001 0.001 0.001"/>
         </geometry>
         <origin xyz="0 0 0.031" rpy="0 0 ${3*PI/2}"/>
@@ -29,11 +29,10 @@
     <gazebo reference="${name}">
         <sensor name="laser" type="ray">
-        <pose>0 0 0 0 0 0</pose>
           <ray>
             <scan>
               <horizontal>
                 <resolution>1</resolution>
-                <max_angle>${PI/2}</max_angle>
-                <min_angle>${PI/2}</min_angle>
+                <max_angle>${3*PI/2}</max_angle>
+                <min_angle>${3*PI/2}</min_angle>
                 <samples>1</samples>
               </horizontal>
@@ -41,7 +40,12 @@
             <range>
               <min>0.08</min>
-              <max>1</max>
+              <max>1.0</max>
               <resolution>0.01</resolution>
             </range>
+            <noise>
+              <type>gaussian</type>
+              <mean>0.0</mean>
+              <stddev>0.01</stddev>
+            </noise>
           </ray>
           <plugin name="laser" filename="libgazebo_ros_laser.so" >
@@ -49,8 +53,11 @@
             <topicName>${name}/scan</topicName>
             <frameName>${name}</frameName>
+            <always_on>1</always_on>
+            <update_rate>60</update_rate>
+            <gaussianNoise>0.005</gaussianNoise>
+            <fov>0</fov>
           </plugin>
-          <always_on>1</always_on>
-          <update_rate>30</update_rate>
           <visualize>true</visualize>
+<!--          <radiation>infrared</radiation>-->
         </sensor>
     </gazebo>

File: urdf/ximea.xacro (robot description, xacro)
@@ -5,14 +5,11 @@
     <link name="${name}">
       <collision>
-        <origin xyz="0 0 0" rpy="0 0 0"/>
+        <origin xyz="-0.037 0 0" rpy="0 ${-PI/2} 0"/>
         <geometry>
-          <box size="0.05 0.05 0.07"/>
+          <cylinder radius="0.0175" length="0.077"/>
         </geometry>
       </collision>
       <visual>
-          <geometry>
-            <box size="0.05 0.05 0.07"/>
-          </geometry>-->
-        <origin xyz="0 0 0" rpy="0 0 0"/>
+        <origin xyz="0 0 0" rpy="${-PI} ${-PI/2} ${-PI}"/>
         <geometry>
           <mesh filename="package://drive_gazebo_sim/meshes/MainCamera.dae" scale="0.001 0.001 0.001"/>
@@ -31,4 +28,46 @@
       <child link="${name}"/>
     </joint>
+<!-- camera -->
+ <gazebo reference="${name}">
+   <sensor type="camera" name="${name}">
+     <update_rate>30.0</update_rate>
+     <camera name="head">
+       <!-- 94 degrees with SY110 lens -->
+       <horizontal_fov>${PI*94/180}</horizontal_fov>
+       <image>
+         <width>2048</width>
+         <height>1088</height>
+         <format>L8</format>
+<!--         <format>R8G8B8</format>-->
+       </image>
+       <clip>
+         <near>0.02</near>
+         <far>300</far>
+       </clip>
+       <noise>
+         <type>gaussian</type>
+         <!-- Noise is sampled independently per pixel on each frame.
+              That pixel's noise value is added to each of its color
+              channels, which at that point lie in the range [0,1]. -->
+         <mean>0.0</mean>
+         <stddev>0.007</stddev>
+       </noise>
+     </camera>
+     <plugin name="camera_controller" filename="libgazebo_ros_camera.so">
+       <alwaysOn>true</alwaysOn>
+       <updateRate>60.0</updateRate>
+       <cameraName>camera</cameraName>
+       <imageTopicName>image_raw</imageTopicName>
+       <cameraInfoTopicName>camera_info</cameraInfoTopicName>
+       <frameName>${name}</frameName>
+       <!-- we do not undistort the ximea camera -->
+       <distortionK1>0.0</distortionK1>
+       <distortionK2>0.0</distortionK2>
+       <distortionK3>0.0</distortionK3>
+       <distortionT1>0.0</distortionT1>
+       <distortionT2>0.0</distortionT2>
+     </plugin>
+   </sensor>
+ </gazebo>
 </xacro:macro>
 </robot>
