Commit message: Usable mass and inertia values, clean up launch files and macros

File: urdf/cc2019.xacro (robot description, xacro)
@@ -3,7 +3,7 @@
     <!-- Import macros -->
     <xacro:include filename="$(find realsense_gazebo_plugin)/urdf/realsense-D435.macro.xacro" />
-    <xacro:include filename="$(find drive_gazebo_sim)/urdf/hokuyo.xacro"/>
-    <xacro:include filename="$(find drive_gazebo_sim)/urdf/pepperl_fuchs_ml100_8_1000_RT.xacro"/>
-    <xacro:include filename="$(find drive_gazebo_sim)/urdf/ximea.xacro"/>
+    <xacro:include filename="$(find drive_gazebo_sim)/urdf/hokuyo_urg04lx.macro.xacro"/>
+    <xacro:include filename="$(find drive_gazebo_sim)/urdf/pepperl_fuchs_ml100_8_1000_RT.macro.xacro"/>
+    <xacro:include filename="$(find drive_gazebo_sim)/urdf/ximea_MQ013MG-ON_SY110.macro.xacro"/>
     <!-- Constants for math -->
     <xacro:property name="PI" value="3.1415926535897931" />
@@ -17,8 +17,8 @@
         <link name="${front_rear}_${right_left}_steer">
             <inertial>
-                <mass value="1.0" />
-                <inertia ixx="1.0" ixy="0.0" ixz="0.0"
-                    iyy="1.0" iyz="0.0"
-                    izz="1.0" />
+                <mass value="0.097624" />
+                <inertia ixx="0.03914" ixy="0.001254" ixz="-0.000188347"
+                    iyy="0.002881" iyz="-0.0008104685"
+                    izz="0.03863" />
             </inertial>
         </link>
@@ -35,5 +35,5 @@
                 <origin rpy="0 ${PI} ${PI/2*(reflect_right_left-1)}" xyz="0 ${-reflect_right_left*length_wheel/2} 0"/>
                 <geometry>
-                    <mesh filename="package://drive_gazebo_sim/meshes/Rad.dae" scale="0.001 0.001 0.001"/>
+                    <mesh filename="package://drive_gazebo_sim/meshes/wheel.dae" scale="0.001 0.001 0.001"/>
                 </geometry>
             </visual>
@@ -107,6 +107,6 @@
      </joint>
     <sensor_hokuyo_urg04lx name="hokuyo" parent="rear_axis_middle" xyz="0.025 0 0.08" rpy="0 0 0"/>
-    <sensor_pepperl_fuchs_ml100_8_1000_RT name="pepperl_fuchs" parent="rear_axis_middle" xyz="0.043 -0.0995 0.021" rpy="0 0 0"/>
-    <sensor_ximea name="ximea" parent="rear_axis_middle" xyz="0.122 0.0 0.233" rpy="${PI} ${-7*PI/6} ${PI}"/>
+    <sensor_pepperl_fuchs_ml100_8_1000_RT name="pepperl_fuchs" parent="rear_axis_middle" xyz="0.043 -0.0995 0.021" rpy="0 0 ${3*PI/2}"/>
+    <sensor_ximea_MQ013MG-ON_SY110 name="ximea" parent="rear_axis_middle" xyz="0.122 0.0 0.233" rpy="${PI} ${-7*PI/6} ${PI}"/>
     <realsense-d435 prefix="realsense" parent="rear_axis_middle">
           <origin xyz="0.02 0 0.105" rpy="0 0 0"/>

Commit message: Add collision mesh for the car body

File: urdf/cc2019.xacro (robot description, xacro)
@@ -93,12 +93,16 @@
         <origin rpy="0 0 ${PI}" xyz="0 0 0" />
         <geometry>
-          <mesh filename="package://drive_gazebo_sim/meshes/Car_reduced.dae" scale="0.001 0.001 0.001"/>
+          <mesh filename="package://drive_gazebo_sim/meshes/hull.dae" scale="0.001 0.001 0.001"/>
         </geometry>
       </visual>
       <collision>
-        <origin rpy="0 0 0" xyz="0.125 0 0.035" />
+        <origin rpy="0 0 0" xyz="0 0 0" />
+        <geometry>
+          <mesh filename="package://drive_gazebo_sim/meshes/hull_collision.dae" scale="0.001 0.001 0.001"/>
+        </geometry>
+<!--        <origin rpy="0 0 0" xyz="0.125 0 0.035" />
         <geometry>
           <box size="0.35 0.2 0.055"/>
-        </geometry>
+        </geometry>-->
       </collision>
       <inertial>
@@ -113,5 +117,5 @@
        <child link="rear_axis_middle"/>
      </joint>
-    <sensor_hokuyo_urg04lx name="hokuyo" parent="rear_axis_middle" xyz="0.025 0 0.08" rpy="0 0 0"/>
+    <sensor_hokuyo_urg04lx name="hokuyo" parent="rear_axis_middle" xyz="0.025 0 0.09" rpy="0 0 0"/>
     <sensor_pepperl_fuchs_ml100_8_1000_RT name="pepperl_fuchs" parent="rear_axis_middle" xyz="0.043 -0.0995 0.021" rpy="0 0 ${3*PI/2}"/>
     <sensor_ximea_MQ013MG-ON_SY110 name="ximea" parent="rear_axis_middle" xyz="0.122 0.0 0.233" rpy="${PI} ${-7*PI/6} ${PI}"/>

Commit message: Add empty world with removed friction for controller testing, sensible controller settings for steering, move to effort controllers

File: urdf/cc2019.xacro (robot description, xacro)
@@ -27,6 +27,6 @@
             <child link="${front_rear}_${right_left}_steer"/>
             <origin xyz="${x_distance} ${-reflect_right_left*length_from_base_to_wheel_y} ${radius_wheel}"/>
-            <dynamics damping="0.7" friction="0.7"/>
-            <limit effort="7.0" lower="${-80*PI/180}" upper="${80*PI/180}" velocity="${200.0*PI/180.0*0.95}"/>
+            <dynamics damping="5" friction="5"/>
+            <limit effort="7" lower="${-80*PI/180}" upper="${80*PI/180}" velocity="200000000"/> <!--velocity="${20*PI*length_wheel}"/>-->
         </joint>
         <link name="${front_rear}_${right_left}_wheel">
@@ -42,4 +42,22 @@
                     <cylinder length="${length_wheel}" radius="${radius_wheel}"/>
                 </geometry>
+                <surface>
+                  <friction>
+                    <ode>
+                      <!-- approximate rubber on track -->
+    <!--                  <mu>0.8</mu>-->
+                        <mu>800.0</mu>
+                        <mu2>600.0</mu2>
+                    </ode>
+                  </friction>
+                  <contact>
+                    <ode>
+                    <kp>1000000.000000</kp>
+                    <kd>1.000000</kd>
+<!--                    <max_vel>100.000000</max_vel>-->
+                    <min_depth>0.00100</min_depth>
+                    </ode>
+                  </contact>
+                </surface>
             </collision>
             <inertial>
@@ -49,12 +67,4 @@
                     izz="0.00003704" />
             </inertial>
-            <surface>
-              <friction>
-                <ode>
-                  <!-- approximate rubber on track -->
-                  <mu>0.8</mu>
-                </ode>
-              </friction>
-            </surface>
         </link>
         <joint name="steer_to_${front_rear}_${right_left}_wheel" type="continuous">
@@ -63,4 +73,6 @@
             <child link="${front_rear}_${right_left}_wheel"/>
             <origin xyz="0 0 0"/>
+            <dynamics damping="5" friction="0"/>
+<!--            <limit effort="0.2" velocity="${6000.0*PI/180.0*radius_wheel}"/>-->
         </joint>
         <!-- Steering transmission -->
@@ -68,8 +80,8 @@
             <type>transmission_interface/SimpleTransmission</type>
             <joint name="chassis_to_${front_rear}_${right_left}_steer">
-                <hardwareInterface>hardware_interface/PositionJointInterface</hardwareInterface>
+                <hardwareInterface>hardware_interface/EffortJointInterface</hardwareInterface>
             </joint>
             <actuator name="${front_rear}_${right_left}_steer">
-                <hardwareInterface>hardware_interface/PositionJointInterface</hardwareInterface>
+                <hardwareInterface>hardware_interface/EffortJointInterface</hardwareInterface>
                 <mechanicalReduction>1</mechanicalReduction>
             </actuator>
@@ -79,8 +91,8 @@
             <type>transmission_interface/SimpleTransmission</type>
             <joint name="steer_to_${front_rear}_${right_left}_wheel">
-                <hardwareInterface>hardware_interface/VelocityJointInterface</hardwareInterface>
+                <hardwareInterface>hardware_interface/EffortJointInterface</hardwareInterface>
             </joint>
             <actuator name="${front_rear}_${right_left}_wheel">
-                <hardwareInterface>hardware_interface/VelocityJointInterface</hardwareInterface>
+                <hardwareInterface>hardware_interface/EffortJointInterface</hardwareInterface>
                 <mechanicalReduction>1</mechanicalReduction>
             </actuator>
@@ -117,10 +129,10 @@
        <child link="rear_axis_middle"/>
      </joint>
-    <sensor_hokuyo_urg04lx name="hokuyo" parent="rear_axis_middle" xyz="0.025 0 0.09" rpy="0 0 0"/>
+<!--    <sensor_hokuyo_urg04lx name="hokuyo" parent="rear_axis_middle" xyz="0.025 0 0.09" rpy="0 0 0"/>
     <sensor_pepperl_fuchs_ml100_8_1000_RT name="pepperl_fuchs" parent="rear_axis_middle" xyz="0.043 -0.0995 0.021" rpy="0 0 ${3*PI/2}"/>
     <sensor_ximea_MQ013MG-ON_SY110 name="ximea" parent="rear_axis_middle" xyz="0.122 0.0 0.233" rpy="${PI} ${-7*PI/6} ${PI}"/>
     <realsense-d435 prefix="realsense" parent="rear_axis_middle">
           <origin xyz="0.02 0 0.105" rpy="0 0 0"/>
-    </realsense-d435>
+    </realsense-d435>-->
     <xacro:steered_wheel right_left="right" reflect_right_left="1" front_rear="front" x_distance="0.22"/>
     <xacro:steered_wheel right_left="left" reflect_right_left="-1" front_rear="front" x_distance="0.22"/>

Commit message: Correctly working steering, fixed inertia of steering link, disabled vel controllers currently

File: urdf/cc2019.xacro (robot description, xacro)
@@ -17,7 +17,10 @@
             <inertial>
                 <mass value="0.097624" />
-                <inertia ixx="0.03914" ixy="0.001254" ixz="-0.000188347"
+<!--                <inertia ixx="0.03914" ixy="0.001254" ixz="-0.000188347"
                     iyy="0.002881" iyz="-0.0008104685"
-                    izz="0.03863" />
+                    izz="0.03863" />-->
+                    <inertia ixx="0.000391" ixy="0.00001125" ixz="0.0"
+                        iyy="0.00002881" iyz="0.0"
+                        izz="0.0003863" />
             </inertial>
         </link>
@@ -27,6 +30,6 @@
             <child link="${front_rear}_${right_left}_steer"/>
             <origin xyz="${x_distance} ${-reflect_right_left*length_from_base_to_wheel_y} ${radius_wheel}"/>
-            <dynamics damping="5" friction="5"/>
-            <limit effort="7" lower="${-80*PI/180}" upper="${80*PI/180}" velocity="200000000"/> <!--velocity="${20*PI*length_wheel}"/>-->
+            <dynamics damping="0.01" friction="0.0"/>
+            <limit effort="1.0" lower="${-80*PI/180}" upper="${80*PI/180}" velocity="200000000"/> <!--velocity="${20*PI*length_wheel}"/>-->
         </joint>
         <link name="${front_rear}_${right_left}_wheel">
@@ -42,28 +45,13 @@
                     <cylinder length="${length_wheel}" radius="${radius_wheel}"/>
                 </geometry>
-                <surface>
-                  <friction>
-                    <ode>
-                      <!-- approximate rubber on track -->
-    <!--                  <mu>0.8</mu>-->
-                        <mu>800.0</mu>
-                        <mu2>600.0</mu2>
-                    </ode>
-                  </friction>
-                  <contact>
-                    <ode>
-                    <kp>1000000.000000</kp>
-                    <kd>1.000000</kd>
-<!--                    <max_vel>100.000000</max_vel>-->
-                    <min_depth>0.00100</min_depth>
-                    </ode>
-                  </contact>
-                </surface>
             </collision>
             <inertial>
                 <mass value="0.049602" />
-                <inertia ixx="0.0000285" ixy="6.01*e-10" ixz="6.691*1e-16"
+<!--                <inertia ixx="0.0000285" ixy="6.01*e-10" ixz="6.691*1e-16"
                     iyy="0.00002853" iyz="3.525*1e-16"
-                    izz="0.00003704" />
+                    izz="0.00003704" />-->
+                    <inertia ixx="0.0000285" ixy="0.0" ixz="0.0"
+                        iyy="0.00002853" iyz="0.0"
+                        izz="0.00003704" />
             </inertial>
         </link>
@@ -73,6 +61,6 @@
             <child link="${front_rear}_${right_left}_wheel"/>
             <origin xyz="0 0 0"/>
-            <dynamics damping="5" friction="0"/>
-<!--            <limit effort="0.2" velocity="${6000.0*PI/180.0*radius_wheel}"/>-->
+            <dynamics damping="0.01" friction="0.0"/>
+            <limit effort="1.0" velocity="${6000.0*PI/180.0*radius_wheel}"/>
         </joint>
         <!-- Steering transmission -->
@@ -98,4 +86,11 @@
             </actuator>
         </transmission>
+        <gazebo reference="${front_rear}_${right_left}_wheel">
+            <mu1 value="1.0"/>
+            <mu2 value="1.0"/>
+            <kp value="10000000.0" />
+            <kd value="1.0" />
+            <fdir1 value="1 0 0"/>
+        </gazebo>
     </xacro:macro>
     <!-- Robot -->
@@ -120,5 +115,5 @@
       <inertial>
           <mass value="2.051134" />
-          <inertia ixx="0.01125" ixy="-0.0008344" ixz="0.008425"
+          <inertia ixx="0.01125" ixy="0.0008344" ixz="0.008425"
               iyy="0.04637" iyz="0.00007786"
               izz="0.0449" />
@@ -129,10 +124,10 @@
        <child link="rear_axis_middle"/>
      </joint>
-<!--    <sensor_hokuyo_urg04lx name="hokuyo" parent="rear_axis_middle" xyz="0.025 0 0.09" rpy="0 0 0"/>
+    <sensor_hokuyo_urg04lx name="hokuyo" parent="rear_axis_middle" xyz="0.025 0 0.09" rpy="0 0 0"/>
     <sensor_pepperl_fuchs_ml100_8_1000_RT name="pepperl_fuchs" parent="rear_axis_middle" xyz="0.043 -0.0995 0.021" rpy="0 0 ${3*PI/2}"/>
     <sensor_ximea_MQ013MG-ON_SY110 name="ximea" parent="rear_axis_middle" xyz="0.122 0.0 0.233" rpy="${PI} ${-7*PI/6} ${PI}"/>
     <realsense-d435 prefix="realsense" parent="rear_axis_middle">
           <origin xyz="0.02 0 0.105" rpy="0 0 0"/>
-    </realsense-d435>-->
+    </realsense-d435>
     <xacro:steered_wheel right_left="right" reflect_right_left="1" front_rear="front" x_distance="0.22"/>
     <xacro:steered_wheel right_left="left" reflect_right_left="-1" front_rear="front" x_distance="0.22"/>

Commit message: Move back to velocity controllers, default settings used, some inertia adjustments

File: urdf/cc2019.xacro (robot description, xacro)
@@ -79,8 +79,8 @@
             <type>transmission_interface/SimpleTransmission</type>
             <joint name="steer_to_${front_rear}_${right_left}_wheel">
-                <hardwareInterface>hardware_interface/EffortJointInterface</hardwareInterface>
+                <hardwareInterface>hardware_interface/VelocityJointInterface</hardwareInterface>
             </joint>
             <actuator name="${front_rear}_${right_left}_wheel">
-                <hardwareInterface>hardware_interface/EffortJointInterface</hardwareInterface>
+                <hardwareInterface>hardware_interface/VelocityJointInterface</hardwareInterface>
                 <mechanicalReduction>1</mechanicalReduction>
             </actuator>

File: urdf/hokuyo_urg04lx_mechanical.macro.xacro (robot description, xacro)
@@ -19,5 +19,5 @@
         <origin xyz="0 0 0" rpy="0 0 0"/>
         <!-- inertia values are not fully correct, but should be close enough for this -->
-        <inertia ixx="0.001505" ixy="-1.89196*1e-7" ixz="-7.5*1e-10" iyy="0.001498" iyz="-0.00001826" izz="0.000368" />
+        <inertia ixx="0.001505" ixy="1.89196*1e-7" ixz="7.5*1e-10" iyy="0.001498" iyz="0.00001826" izz="0.000368" />
       </inertial>
     </link>

File: urdf/pepperl_fuchs_ml100_8_1000_RT.macro.xacro (robot description, xacro)
@@ -19,5 +19,5 @@
         <origin xyz="0 0 0" rpy="0 0 0"/>
         <!-- inertia values are approximate but should be close enough -->
-        <inertia ixx="0.00001784" ixy="0.0000026951" ixz="-0.0000073832" iyy="0.0000226" iyz="0.0000042295" izz="0.0000013921" />
+        <inertia ixx="0.00001784" ixy="0.0000026951" ixz="0.0000073832" iyy="0.0000226" iyz="0.0000042295" izz="0.0000013921" />
       </inertial>
     </link>

File: urdf/ximea_MQ013MG-ON_SY110.macro.xacro (robot description, xacro)
@@ -21,5 +21,5 @@
         <origin xyz="0 0 0" rpy="0 0 0"/>
         <!-- inertia values are approximate but should be close enough -->
-        <inertia ixx="0.0009728102" ixy="0.0000950064" ixz="0.0000154579" iyy="0.01061" iyz="-7.4781e-7" izz="0.01062" />
+        <inertia ixx="0.0009728102" ixy="0.0000950064" ixz="0.0000154579" iyy="0.0001061" iyz="-7.4781e-7" izz="0.0001062" />
       </inertial>
     </link>

Commit message: Add materials to car, wheels, ximea, pepperl_fuchs

File: urdf/cc2019.xacro (robot description, xacro)
@@ -35,7 +35,7 @@
         <link name="${front_rear}_${right_left}_wheel">
             <visual>
-                <origin rpy="0 ${PI} ${PI/2*(reflect_right_left-1)}" xyz="0 ${-reflect_right_left*length_wheel/2} 0"/>
+                <origin rpy="${PI/2} ${PI} ${PI/2*(reflect_right_left-1)}" xyz="0 ${-reflect_right_left*length_wheel/2} 0"/>
                 <geometry>
-                    <mesh filename="package://drive_gazebo_sim/meshes/wheel.dae" scale="0.001 0.001 0.001"/>
+                    <mesh filename="package://drive_gazebo_sim/meshes/wheel.dae" scale="1 1 1"/>
                 </geometry>
             </visual>
@@ -100,5 +100,5 @@
         <origin rpy="0 0 ${PI}" xyz="0 0 0" />
         <geometry>
-          <mesh filename="package://drive_gazebo_sim/meshes/hull.dae" scale="0.001 0.001 0.001"/>
+          <mesh filename="package://drive_gazebo_sim/meshes/hull.dae" scale="1 1 1"/>
         </geometry>
       </visual>

File: urdf/pepperl_fuchs_ml100_8_1000_RT.macro.xacro (robot description, xacro)
@@ -11,5 +11,5 @@
       <visual>
         <geometry>
-          <mesh filename="package://drive_gazebo_sim/meshes/pepperl_fuchs_ml100.dae" scale="0.001 0.001 0.001"/>
+          <mesh filename="package://drive_gazebo_sim/meshes/pepperl_fuchs_ml100.dae" scale="1 1 1"/>
         </geometry>
         <origin xyz="0 0 0.031" rpy="0 0 0"/>

File: urdf/ximea_MQ013MG-ON_SY110.macro.xacro (robot description, xacro)
@@ -13,5 +13,5 @@
         <origin xyz="0 0 0" rpy="0 0 0"/>
         <geometry>
-          <mesh filename="package://drive_gazebo_sim/meshes/ximea_MQ013MG-ON_SY110.dae" scale="0.001 0.001 0.001"/>
+          <mesh filename="package://drive_gazebo_sim/meshes/ximea_MQ013MG-ON_SY110.dae" scale="1 1 1"/>
         </geometry>
       </visual>

Commit message: Move chassis center of mass to correct location

File: urdf/cc2019.xacro (robot description, xacro)
@@ -113,10 +113,4 @@
         </geometry>-->
       </collision>
-      <inertial>
-          <mass value="2.051134" />
-          <inertia ixx="0.01125" ixy="0.0008344" ixz="0.008425"
-              iyy="0.04637" iyz="0.00007786"
-              izz="0.0449" />
-      </inertial>
     </link>
     <joint name="base_joint" type="fixed">
@@ -124,4 +118,17 @@
        <child link="rear_axis_middle"/>
      </joint>
+    <joint name="rear_to_chassis" type="fixed">
+       <parent link="rear_axis_middle"/>
+       <child link="chassis"/>
+       <origin xyz="0.110912 0.00420803 0.0422526"/>
+     </joint>
+    <link name="chassis">
+       <inertial>
+          <mass value="2.051134" />
+          <inertia ixx="0.01125" ixy="0.0008344" ixz="0.008425"
+              iyy="0.04637" iyz="0.00007786"
+              izz="0.0449" />
+       </inertial>
+    </link>
     <sensor_hokuyo_urg04lx name="hokuyo" parent="rear_axis_middle" xyz="0.025 0 0.09" rpy="0 0 0"/>
     <sensor_pepperl_fuchs_ml100_8_1000_RT name="pepperl_fuchs" parent="rear_axis_middle" xyz="0.043 -0.0995 0.021" rpy="0 0 ${3*PI/2}"/>
