Commit message: Add scaling, update parameters

File: urdf/cc2019.xacro (robot description, xacro)
@@ -12,14 +12,33 @@
     <xacro:property name="radius_wheel" value="0.032" />
     <xacro:property name="length_from_base_to_wheel_y" value="0.088" />
+    <xacro:property name="steering_offset" value="0.05" />
+    <xacro:property name="mass_scaling_factor" value="10000" />
+    <xacro:property name="inertia_scaling_factor" value="10000" />
+    <xacro:macro name="scaled_mass" params="value">
+        <mass value="${value * mass_scaling_factor}" />
+    </xacro:macro>
+    <xacro:macro name="scaled_inertia" params="ixx ixy ixz iyy iyz izz">
+        <inertia
+            ixx="${ixx * inertia_scaling_factor}"
+            ixy="${ixy * inertia_scaling_factor}"
+            ixz="${ixz * inertia_scaling_factor}"
+            iyy="${iyy * inertia_scaling_factor}"
+            iyz="${iyz * inertia_scaling_factor}"
+            izz="${izz * inertia_scaling_factor}" />
+    </xacro:macro>
    <!-- Wheel macro -->
    <xacro:macro name="steered_wheel" params="right_left reflect_right_left front_rear x_distance">
         <link name="${front_rear}_${right_left}_steer">
             <inertial>
-                <mass value="0.097624" />
+                <xacro:scaled_mass value="0.097624" />
 <!--                <inertia ixx="0.03914" ixy="0.001254" ixz="-0.000188347"
                     iyy="0.002881" iyz="-0.0008104685"
                     izz="0.03863" />-->
-                    <inertia ixx="0.000391" ixy="0.00001125" ixz="0.0"
-                        iyy="0.00002881" iyz="0.0"
+                    <xacro:scaled_inertia
+                        ixx="0.000391"
+                        ixy="0.00001125"
+                        ixz="0.0"
+                        iyy="0.00002881"
+                        iyz="0.0"
                         izz="0.0003863" />
             </inertial>
@@ -29,5 +48,5 @@
             <parent link="rear_axis_middle"/>
             <child link="${front_rear}_${right_left}_steer"/>
-            <origin xyz="${x_distance} ${-reflect_right_left*length_from_base_to_wheel_y} ${radius_wheel}"/>
+            <origin xyz="${x_distance} ${-reflect_right_left * (length_from_base_to_wheel_y - steering_offset)} ${radius_wheel}"/>
             <dynamics damping="0.01" friction="0.0"/>
             <limit effort="1.0" lower="${-80*PI/180}" upper="${80*PI/180}" velocity="200000000"/> <!--velocity="${20*PI*length_wheel}"/>-->
@@ -47,9 +66,9 @@
             </collision>
             <inertial>
-                <mass value="0.049602" />
+                <xacro:scaled_mass value="0.049602" />
 <!--                <inertia ixx="0.0000285" ixy="6.01*e-10" ixz="6.691*1e-16"
                     iyy="0.00002853" iyz="3.525*1e-16"
                     izz="0.00003704" />-->
-                    <inertia ixx="0.0000285" ixy="0.0" ixz="0.0"
+                    <xacro:scaled_inertia ixx="0.0000285" ixy="0.0" ixz="0.0"
                         iyy="0.00002853" iyz="0.0"
                         izz="0.00003704" />
@@ -60,5 +79,5 @@
             <parent link="${front_rear}_${right_left}_steer"/>
             <child link="${front_rear}_${right_left}_wheel"/>
-            <origin xyz="0 0 0"/>
+            <origin xyz="0 ${-reflect_right_left * steering_offset} 0"/>
             <dynamics damping="0.01" friction="0.0"/>
             <limit effort="1.0" velocity="${6000.0*PI/180.0*radius_wheel}"/>
@@ -76,21 +95,21 @@
         </transmission>
         <!-- Wheel transmission -->
-        <transmission name="tran_wheel_${front_rear}_${right_left}">
+<!--        <transmission name="tran_wheel_${front_rear}_${right_left}">
             <type>transmission_interface/SimpleTransmission</type>
             <joint name="steer_to_${front_rear}_${right_left}_wheel">
-                <hardwareInterface>hardware_interface/VelocityJointInterface</hardwareInterface>
+                <hardwareInterface>hardware_interface/EffortJointInterface</hardwareInterface>
             </joint>
             <actuator name="${front_rear}_${right_left}_wheel">
-                <hardwareInterface>hardware_interface/VelocityJointInterface</hardwareInterface>
+                <hardwareInterface>hardware_interface/EffortJointInterface</hardwareInterface>
                 <mechanicalReduction>1</mechanicalReduction>
             </actuator>
-        </transmission>
-        <gazebo reference="${front_rear}_${right_left}_wheel">
+        </transmission>-->
+<!--        <gazebo reference="${front_rear}_${right_left}_wheel">
             <mu1 value="1.0"/>
             <mu2 value="1.0"/>
-            <kp value="10000000.0" />
+            <kp value="10.0" />
             <kd value="1.0" />
             <fdir1 value="1 0 0"/>
-        </gazebo>
+        </gazebo>-->
     </xacro:macro>
     <!-- Robot -->
@@ -125,16 +144,16 @@
     <link name="chassis">
        <inertial>
-          <mass value="2.051134" />
-          <inertia ixx="0.01125" ixy="0.0008344" ixz="0.008425"
+          <xacro:scaled_mass value="2.051134" />
+          <xacro:scaled_inertia ixx="0.01125" ixy="0.0008344" ixz="0.008425"
               iyy="0.04637" iyz="0.00007786"
               izz="0.0449" />
        </inertial>
     </link>
-    <sensor_hokuyo_urg04lx name="hokuyo" parent="rear_axis_middle" xyz="0.025 0 0.09" rpy="0 0 0"/>
+<!--    <sensor_hokuyo_urg04lx name="hokuyo" parent="rear_axis_middle" xyz="0.025 0 0.09" rpy="0 0 0"/>
     <sensor_pepperl_fuchs_ml100_8_1000_RT name="pepperl_fuchs" parent="rear_axis_middle" xyz="0.043 -0.0995 0.021" rpy="0 0 ${3*PI/2}"/>
     <sensor_ximea_MQ013MG-ON_SY110 name="ximea" parent="rear_axis_middle" xyz="0.122 0.0 0.233" rpy="${PI} ${-7*PI/6} ${PI}"/>
     <realsense-d435 prefix="realsense" parent="rear_axis_middle">
           <origin xyz="0.02 0 0.105" rpy="0 0 0"/>
-    </realsense-d435>
+    </realsense-d435>-->
     <xacro:steered_wheel right_left="right" reflect_right_left="1" front_rear="front" x_distance="0.22"/>
     <xacro:steered_wheel right_left="left" reflect_right_left="-1" front_rear="front" x_distance="0.22"/>

Commit message: Working steering controllers

File: urdf/cc2019.xacro (robot description, xacro)
@@ -13,6 +13,6 @@
     <xacro:property name="length_from_base_to_wheel_y" value="0.088" />
     <xacro:property name="steering_offset" value="0.05" />
-    <xacro:property name="mass_scaling_factor" value="10000" />
-    <xacro:property name="inertia_scaling_factor" value="10000" />
+    <xacro:property name="mass_scaling_factor" value="10" />
+    <xacro:property name="inertia_scaling_factor" value="100" />
     <xacro:macro name="scaled_mass" params="value">
         <mass value="${value * mass_scaling_factor}" />
@@ -95,5 +95,5 @@
         </transmission>
         <!-- Wheel transmission -->
-<!--        <transmission name="tran_wheel_${front_rear}_${right_left}">
+        <transmission name="tran_wheel_${front_rear}_${right_left}">
             <type>transmission_interface/SimpleTransmission</type>
             <joint name="steer_to_${front_rear}_${right_left}_wheel">
@@ -104,5 +104,5 @@
                 <mechanicalReduction>1</mechanicalReduction>
             </actuator>
-        </transmission>-->
+        </transmission>
 <!--        <gazebo reference="${front_rear}_${right_left}_wheel">
             <mu1 value="1.0"/>

Commit message: Working controller setup, however very high command efforts currently and physical values upscaled to prevent gazebo errors

File: urdf/cc2019.xacro (robot description, xacro)
@@ -50,5 +50,5 @@
             <origin xyz="${x_distance} ${-reflect_right_left * (length_from_base_to_wheel_y - steering_offset)} ${radius_wheel}"/>
             <dynamics damping="0.01" friction="0.0"/>
-            <limit effort="1.0" lower="${-80*PI/180}" upper="${80*PI/180}" velocity="200000000"/> <!--velocity="${20*PI*length_wheel}"/>-->
+            <limit effort="10.0" lower="${-80*PI/180}" upper="${80*PI/180}" velocity="200000000"/> <!--velocity="${20*PI*length_wheel}"/>-->
         </joint>
         <link name="${front_rear}_${right_left}_wheel">
@@ -70,7 +70,7 @@
                     iyy="0.00002853" iyz="3.525*1e-16"
                     izz="0.00003704" />-->
-                    <xacro:scaled_inertia ixx="0.0000285" ixy="0.0" ixz="0.0"
-                        iyy="0.00002853" iyz="0.0"
-                        izz="0.00003704" />
+                    <xacro:scaled_inertia ixx="0.000285" ixy="0.0" ixz="0.0"
+                        iyy="0.0002853" iyz="0.0"
+                        izz="0.0003704" />
             </inertial>
         </link>
@@ -150,10 +150,10 @@
        </inertial>
     </link>
-<!--    <sensor_hokuyo_urg04lx name="hokuyo" parent="rear_axis_middle" xyz="0.025 0 0.09" rpy="0 0 0"/>
+    <sensor_hokuyo_urg04lx name="hokuyo" parent="rear_axis_middle" xyz="0.025 0 0.09" rpy="0 0 0"/>
     <sensor_pepperl_fuchs_ml100_8_1000_RT name="pepperl_fuchs" parent="rear_axis_middle" xyz="0.043 -0.0995 0.021" rpy="0 0 ${3*PI/2}"/>
     <sensor_ximea_MQ013MG-ON_SY110 name="ximea" parent="rear_axis_middle" xyz="0.122 0.0 0.233" rpy="${PI} ${-7*PI/6} ${PI}"/>
     <realsense-d435 prefix="realsense" parent="rear_axis_middle">
           <origin xyz="0.02 0 0.105" rpy="0 0 0"/>
-    </realsense-d435>-->
+    </realsense-d435>
     <xacro:steered_wheel right_left="right" reflect_right_left="1" front_rear="front" x_distance="0.22"/>
     <xacro:steered_wheel right_left="left" reflect_right_left="-1" front_rear="front" x_distance="0.22"/>

Commit message: Controller tuning to allow higher driving speeds

File: urdf/cc2019.xacro (robot description, xacro)
@@ -81,5 +81,5 @@
             <origin xyz="0 ${-reflect_right_left * steering_offset} 0"/>
             <dynamics damping="0.01" friction="0.0"/>
-            <limit effort="1.0" velocity="${6000.0*PI/180.0*radius_wheel}"/>
+            <limit effort="1.0" velocity="${60000.0*PI/180.0*radius_wheel}"/>
         </joint>
         <!-- Steering transmission -->

Commit message: Move camera origin to sensor

File: urdf/cc2019.xacro (robot description, xacro)
@@ -152,5 +152,5 @@
     <sensor_hokuyo_urg04lx name="hokuyo" parent="rear_axis_middle" xyz="0.025 0 0.09" rpy="0 0 0"/>
     <sensor_pepperl_fuchs_ml100_8_1000_RT name="pepperl_fuchs" parent="rear_axis_middle" xyz="0.043 -0.0995 0.021" rpy="0 0 ${3*PI/2}"/>
-    <sensor_ximea_MQ013MG-ON_SY110 name="ximea" parent="rear_axis_middle" xyz="0.122 0.0 0.233" rpy="${PI} ${-7*PI/6} ${PI}"/>
+    <sensor_ximea_MQ013MG-ON_SY110 name="ximea" parent="rear_axis_middle" xyz="0.085 0.0 0.255" rpy="${PI} ${-7*PI/6} ${PI}"/>
     <realsense-d435 prefix="realsense" parent="rear_axis_middle">
           <origin xyz="0.02 0 0.105" rpy="0 0 0"/>

File: urdf/ximea_MQ013MG-ON_SY110.macro.xacro (robot description, xacro)
@@ -11,5 +11,5 @@
       </collision>
       <visual>
-        <origin xyz="0 0 0" rpy="0 0 0"/>
+        <origin xyz="0.037 0 0" rpy="0 0 0"/>
         <geometry>
           <mesh filename="package://drive_gazebo_sim/meshes/ximea_MQ013MG-ON_SY110.dae" scale="1 1 1"/>
@@ -45,5 +45,5 @@
        </image>
        <clip>
-         <near>0.02</near>
+         <near>0.05</near>
          <far>300</far>
        </clip>
@@ -71,4 +71,5 @@
        <distortionT2>0.0</distortionT2>
      </plugin>
+     <visualize>1</visualize>
    </sensor>
  </gazebo>
